File: Schema2/schema2.sch (EAGLE design)
At the start: 34 parts, among them IC1 LM2596S, IC2 78L05CPK, IC3 TL431ACDBZ, IC4 LM358D, X1 22-23-2021, X2 22-23-2021

Commit message: update schema
Parts:
- removed PAD1, PAD2: (no value), wirepad:2,54/1,0
- removed X2: 22-23-2021, con-molex:22-23-2021
- added C8: 1uF, eagle-ltspice:C
- added R11: 80R, resistor:R-EU_M0805
- added X3: (no value), con-phoenix-254:MPT2
- IC1: value LM2596S -> XL4015; device linear:LM2596S -> moje:XL4015
- X1: value 22-23-2021 -> (none); device con-molex:22-23-2021 -> con-phoenix-254:MPT2
Connections:
- removed net N$8: IC1.EN, PAD1.P
- new net N$4: IC4A.OUT, R11.2
- new net N$5: C8.2, IC1.VC
- net GND: now also IC1.GND; no longer PAD2.P
- net N$1: now also X3-1.1; no longer X1-1.S
- net N$10: now also IC1.SW; no longer IC1.OUT
- net N$11: now also R11.1; no longer IC4A.OUT
- net N$12: now also X1-1.1; no longer X2-1.S
- net N$21: now also X1-2.1; no longer X2-2.S
- net N$3: now also X3-2.1; no longer X1-2.S
- net VCC_IN: now also C8.1
Other:
- moved on the sheet: C5, IC4B, LED1, LED2, LED3, PAD3, PAD4, R1, R10, R5, R6, R7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

Commit message: update schema
Parts:
- removed R10: 0,05R, eagle-ltspice:RR2512
- removed R11: 80R, resistor:R-EU_M0805
- removed X1, X3: (no value), con-phoenix-254:MPT2
- added C9: 1uF, eagle-ltspice:C
- added J1, J2: (no value), con-amp:MTA02-156
- added P1, P2: 10K, pot:TRIM_EU-3223G
- added PAD2, PAD5, PAD6: (no value), wirepad:2,15/1,0
- C1, C2: value 10uF -> (none); device eagle-ltspice:C -> adafruit:CPOL-USE5-10.5
- C3: value 1uF -> 10uF
- C6: value 470uF -> 1uF; device resistor:CPOL-US153CLV-0605 -> eagle-ltspice:C
- C7: value 470uF -> 10uF; device resistor:CPOL-US153CLV-0605 -> eagle-ltspice:C
- C8: value 1uF -> 470uF; device eagle-ltspice:C -> resistor:CPOL-US153CLV-0605
- F1: value (none) -> FUSEGSH15; device fuse:SHK20Q -> fuse:FUSEGSH15
- IC2: value 78L05CPK -> 78L05
- IC3: value TL431ACDBZ -> TL431
- PAD3, PAD4: device wirepad:2,54/1,0 -> wirepad:2,15/1,0
- R1: value 10K -> 2,2K; device pot:TRIM_EU-3223G -> resistor:R-EU_M0805
- R2: value 10K -> 68K; device pot:TRIM_EU-3223G -> resistor:R-EU_M0805
- R3: value 2,2K -> 80R
- R4: value 71,5K -> 100K
- R5: value 270R -> 10K
- R6: value 90,9K -> 270R
- R7: value 10K -> 1K
- R9: value 1K -> 0,05R; device resistor:R-EU_M0805 -> eagle-ltspice:RR2512
- renumbered L2 to L1
Connections:
- removed net N$6: C3.1, IC2.OUT, IC4P.V+, R3.1, R8.1
- new net VNN: C4.1, IC2.OUT, IC4P.V+, R1.1, R7.1
- net GND: now also C1.-, C2.-, C5.2, C7.2, C8.-, P1.A, PAD5.P, R5.2, R6.1, R9.1; no longer C1.2, C2.2, C6.-, C7.-, IC1.GND@1, PAD3.P, R10.1, R2.A, R5.1, R7.2
- net N$1: now also F1.1, J1.2; no longer F1.1A, X3-1.1
- net N$10: now also IC1.SW@1
- net N$11: now also C9.1, R3.1; no longer C5.1, R11.1
- net N$12: now also C7.1, C8.+, J2.1, P2.E, P2.S, PAD3.P; no longer C1.1, C7.+, R1.E, R1.S, X1-1.1
- net N$14: now also P2.A, PAD2.P, R6.2; no longer R1.A, R5.2
- net N$15: now also C5.1, R1.2, R2.1; no longer C4.1, R3.2, R4.1
- net N$16: now also R4.1, R5.1; no longer R6.1, R7.1
- net N$18: now also R8.2; no longer R9.2
- net N$2: now also F1.2; no longer F1.2A
- net N$20: now also R7.2; no longer R8.2
- net N$21: now also J2.2, R8.1, R9.2; no longer PAD4.P, R10.2, R9.1, X1-2.1
- net N$3: now also J1.1; no longer X3-2.1
- net N$4: now also R3.2; no longer R11.2
- net N$5: now also C6.2; no longer C8.2
- net N$7: now also P1.E, PAD4.P, R2.2; no longer R2.E, R4.2
- net N$9: now also C9.2, P1.S, PAD6.P, R4.2; no longer C5.2, R2.S, R6.2
- net VCC_IN: now also C1.+, C2.+, C3.1, C6.1; no longer C2.1, C6.+, C8.1
Other:
- note added: "1,25 - 24 V"
- moved on the sheet: B2, C3, C4, C5, IC1, R3, R4, R5, R6, R7, R8, R9

Commit message: update schema
Parts:
- removed B2: RECTIFIER-KBU, rectifier:RECTIFIER-KBU
- added B1: RECTIFIER-2KBP, rectifier:RECTIFIER-2KBP
- added PAD1, PAD7: (no value), wirepad:2,15/1,0
- C1, C2: value (none) -> 1000uF
Connections:
- net GND: now also B1.-, PAD1.P; no longer B2.-
- net N$2: now also B1.AC1; no longer B2.AC1
- net N$21: now also PAD7.P
- net N$3: now also B1.AC2; no longer B2.AC2
- net VCC_IN: now also B1.+; no longer B2.+
Changed lines of the file:
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@@
 <setting verticaltext="up"/>
 </settings>
-<grid distance="0.1" unitdist="inch" unit="inch" style="lines" multiple="1" display="yes" altdistance="0.01" altunitdist="inch" altunit="inch"/>
+<grid distance="0.1" unitdist="inch" unit="inch" style="lines" multiple="1" display="no" altdistance="0.01" altunitdist="inch" altunit="inch"/>
 <layers>
-<layer number="1" name="Top" color="4" fill="1" visible="yes" active="no"/>
-<layer number="16" name="Bottom" color="1" fill="1" visible="yes" active="no"/>
-<layer number="17" name="Pads" color="2" fill="1" visible="yes" active="no"/>
-<layer number="18" name="Vias" color="2" fill="1" visible="yes" active="no"/>
-<layer number="19" name="Unrouted" color="6" fill="1" visible="yes" active="no"/>
-<layer number="20" name="Dimension" color="15" fill="1" visible="yes" active="no"/>
-<layer number="21" name="tPlace" color="7" fill="1" visible="yes" active="no"/>
-<layer number="22" name="bPlace" color="7" fill="1" visible="yes" active="no"/>
-<layer number="23" name="tOrigins" color="15" fill="1" visible="yes" active="no"/>
-<layer number="24" name="bOrigins" color="15" fill="1" visible="yes" active="no"/>
-<layer number="25" name="tNames" color="7" fill="1" visible="yes" active="no"/>
-<layer number="26" name="bNames" color="7" fill="1" visible="yes" active="no"/>
-<layer number="27" name="tValues" color="7" fill="1" visible="yes" active="no"/>
-<layer number="28" name="bValues" color="7" fill="1" visible="yes" active="no"/>
+<layer number="1" name="Top" color="4" fill="1" visible="no" active="no"/>
+<layer number="16" name="Bottom" color="1" fill="1" visible="no" active="no"/>
+<layer number="17" name="Pads" color="2" fill="1" visible="no" active="no"/>
+<layer number="18" name="Vias" color="2" fill="1" visible="no" active="no"/>
+<layer number="19" name="Unrouted" color="6" fill="1" visible="no" active="no"/>
+<layer number="20" name="Dimension" color="15" fill="1" visible="no" active="no"/>
+<layer number="21" name="tPlace" color="7" fill="1" visible="no" active="no"/>
+<layer number="22" name="bPlace" color="7" fill="1" visible="no" active="no"/>
+<layer number="23" name="tOrigins" color="15" fill="1" visible="no" active="no"/>
+<layer number="24" name="bOrigins" color="15" fill="1" visible="no" active="no"/>
+<layer number="25" name="tNames" color="7" fill="1" visible="no" active="no"/>
+<layer number="26" name="bNames" color="7" fill="1" visible="no" active="no"/>
+<layer number="27" name="tValues" color="7" fill="1" visible="no" active="no"/>
+<layer number="28" name="bValues" color="7" fill="1" visible="no" active="no"/>
 <layer number="29" name="tStop" color="7" fill="3" visible="no" active="no"/>
 <layer number="30" name="bStop" color="7" fill="6" visible="no" active="no"/>
@@
 <layer number="35" name="tGlue" color="7" fill="4" visible="no" active="no"/>
 <layer number="36" name="bGlue" color="7" fill="5" visible="no" active="no"/>
-<layer number="37" name="tTest" color="7" fill="1" visible="yes" active="no"/>
-<layer number="38" name="bTest" color="7" fill="1" visible="yes" active="no"/>
+<layer number="37" name="tTest" color="7" fill="1" visible="no" active="no"/>
+<layer number="38" name="bTest" color="7" fill="1" visible="no" active="no"/>
 <layer number="39" name="tKeepout" color="4" fill="11" visible="no" active="no"/>
 <layer number="40" name="bKeepout" color="1" fill="11" visible="no" active="no"/>
@@
 <layer number="44" name="Drills" color="7" fill="1" visible="no" active="no"/>
 <layer number="45" name="Holes" color="7" fill="1" visible="no" active="no"/>
-<layer number="46" name="Milling" color="3" fill="1" visible="yes" active="no"/>
-<layer number="47" name="Measures" color="7" fill="1" visible="yes" active="no"/>
-<layer number="48" name="Document" color="7" fill="1" visible="yes" active="no"/>
-<layer number="49" name="Reference" color="7" fill="1" visible="yes" active="no"/>
-<layer number="50" name="dxf" color="7" fill="1" visible="yes" active="no"/>
-<layer number="51" name="tDocu" color="7" fill="1" visible="yes" active="no"/>
-<layer number="52" name="bDocu" color="7" fill="1" visible="yes" active="no"/>
-<layer number="53" name="tGND_GNDA" color="7" fill="9" visible="yes" active="no"/>
-<layer number="54" name="bGND_GNDA" color="1" fill="9" visible="yes" active="no"/>
-<layer number="56" name="wert" color="7" fill="1" visible="yes" active="no"/>
-<layer number="57" name="tCAD" color="7" fill="1" visible="yes" active="no"/>
-<layer number="59" name="tCarbon" color="7" fill="1" visible="yes" active="no"/>
-<layer number="60" name="bCarbon" color="7" fill="1" visible="yes" active="no"/>
+<layer number="46" name="Milling" color="3" fill="1" visible="no" active="no"/>
+<layer number="47" name="Measures" color="7" fill="1" visible="no" active="no"/>
+<layer number="48" name="Document" color="7" fill="1" visible="no" active="no"/>
+<layer number="49" name="Reference" color="7" fill="1" visible="no" active="no"/>
+<layer number="50" name="dxf" color="7" fill="1" visible="no" active="no"/>
+<layer number="51" name="tDocu" color="7" fill="1" visible="no" active="no"/>
+<layer number="52" name="bDocu" color="7" fill="1" visible="no" active="no"/>
+<layer number="53" name="tGND_GNDA" color="7" fill="9" visible="no" active="no"/>
+<layer number="54" name="bGND_GNDA" color="1" fill="9" visible="no" active="no"/>
+<layer number="56" name="wert" color="7" fill="1" visible="no" active="no"/>
+<layer number="57" name="tCAD" color="7" fill="1" visible="no" active="no"/>
+<layer number="59" name="tCarbon" color="7" fill="1" visible="no" active="no"/>
+<layer number="60" name="bCarbon" color="7" fill="1" visible="no" active="no"/>
 <layer number="90" name="Modules" color="5" fill="1" visible="yes" active="yes"/>
 <layer number="91" name="Nets" color="2" fill="1" visible="yes" active="yes"/>
@@
 <part name="LED3" library="eagle-ltspice" deviceset="LED_E" device=""/>
 <part name="L1" library="inductors" deviceset="ED16" device="" value="40uH"/>
-<part name="B2" library="rectifier" deviceset="RECTIFIER-" device="KBU"/>
+<part name="B1" library="rectifier" deviceset="RECTIFIER-" device="2KBP" value="RECTIFIER-2KBP"/>
 <part name="R3" library="resistor" deviceset="R-EU_" device="M0805" value="80R"/>
 <part name="C6" library="eagle-ltspice" deviceset="C" device="" value="1uF"/>
@@
 <part name="J2" library="con-amp" deviceset="MTA02-156" device=""/>
 <part name="F1" library="fuse" deviceset="FUSE" device="GSH15"/>
-<part name="C1" library="adafruit" deviceset="CPOL-US" device="E5-10.5"/>
-<part name="C2" library="adafruit" deviceset="CPOL-US" device="E5-10.5"/>
+<part name="C1" library="adafruit" deviceset="CPOL-US" device="E5-10.5" value="1000uF"/>
+<part name="C2" library="adafruit" deviceset="CPOL-US" device="E5-10.5" value="1000uF"/>
 <part name="PAD2" library="wirepad" deviceset="2,15/1,0" device=""/>
 <part name="PAD3" library="wirepad" deviceset="2,15/1,0" device=""/>
@@
 <part name="PAD5" library="wirepad" deviceset="2,15/1,0" device=""/>
 <part name="PAD6" library="wirepad" deviceset="2,15/1,0" device=""/>
+<part name="PAD1" library="wirepad" deviceset="2,15/1,0" device=""/>
+<part name="PAD7" library="wirepad" deviceset="2,15/1,0" device=""/>
 </parts>
 <sheets>
@@
 <instance part="LED3" gate="G$1" x="175.26" y="43.18" rot="R180"/>
 <instance part="L1" gate="1" x="137.16" y="68.58"/>
-<instance part="B2" gate="G$1" x="27.94" y="27.94" smashed="yes">
+<instance part="B1" gate="G$1" x="27.94" y="27.94" smashed="yes">
 <attribute name="NAME" x="33.02" y="30.48" size="1.778" layer="95"/>
 </instance>
@@
 <instance part="PAD5" gate="1" x="132.08" y="-2.54"/>
 <instance part="PAD6" gate="1" x="142.24" y="5.08" rot="R90"/>
+<instance part="PAD1" gate="1" x="205.74" y="-10.16" rot="R90"/>
+<instance part="PAD7" gate="1" x="218.44" y="-10.16" rot="R90"/>
 </instances>
 <busses>
@@
 <wire x1="17.78" y1="38.1" x2="27.94" y2="38.1" width="0.1524" layer="91"/>
 <wire x1="27.94" y1="38.1" x2="27.94" y2="33.02" width="0.1524" layer="91"/>
-<pinref part="B2" gate="G$1" pin="AC1"/>
+<pinref part="B1" gate="G$1" pin="AC1"/>
 <pinref part="F1" gate="G$1" pin="2"/>
 </segment>
@@
 <wire x1="0" y1="17.78" x2="27.94" y2="17.78" width="0.1524" layer="91"/>
 <wire x1="27.94" y1="17.78" x2="27.94" y2="22.86" width="0.1524" layer="91"/>
-<pinref part="B2" gate="G$1" pin="AC2"/>
+<pinref part="B1" gate="G$1" pin="AC2"/>
 <wire x1="0" y1="17.78" x2="0" y2="27.94" width="0.1524" layer="91"/>
 <pinref part="J1" gate="G$1" pin="1"/>
@@
 <junction x="66.04" y="27.94"/>
 <junction x="66.04" y="22.86"/>
-<pinref part="B2" gate="G$1" pin="+"/>
+<pinref part="B1" gate="G$1" pin="+"/>
 <pinref part="C6" gate="G$1" pin="1"/>
 <wire x1="83.82" y1="58.42" x2="83.82" y2="60.96" width="0.1524" layer="91"/>
@@
 <junction x="185.42" y="-7.62"/>
 <junction x="185.42" y="0"/>
-<pinref part="B2" gate="G$1" pin="-"/>
+<pinref part="B1" gate="G$1" pin="-"/>
 <pinref part="C1" gate="G$1" pin="-"/>
 <wire x1="40.64" y1="5.08" x2="40.64" y2="-7.62" width="0.1524" layer="91"/>
@@
 <pinref part="PAD5" gate="1" pin="P"/>
 <junction x="134.62" y="-2.54"/>
+<pinref part="PAD1" gate="1" pin="P"/>
+<junction x="205.74" y="-7.62"/>
 </segment>
 <segment>
@@
 <junction x="198.12" y="22.86"/>
 <pinref part="J2" gate="G$1" pin="2"/>
-</segment>
-</net>
+<pinref part="PAD7" gate="1" pin="P"/>
+</segment>
+</net>
